File: ESP32-DevBoard-Breakout.kicad_sch (KiCad schematic)
At the start: 0 parts

Commit message: Customised schematic template
Other:
- company: (none) -> https://github.com/colinmakerofthings
- title: (none) -> ESP32 Development Board Breakout

Commit message: Added connectors and terminals
Parts:
- added J1, J2: Screw_Terminal_01x15, symbol Connector:Screw_Terminal_01x15
- added J10: Screw_Terminal_01x02, symbol Connector:Screw_Terminal_01x02
- added J11, J3: Conn_01x15_Pin, symbol Connector:Conn_01x15_Pin
- added J12, J4: Conn_01x15_Socket, symbol Connector:Conn_01x15_Socket
- added J5: Conn_01x03_Socket, symbol Connector:Conn_01x03_Socket
- added J6, J7, J8: Conn_01x06_Pin, symbol Connector:Conn_01x06_Pin
- added J9: Conn_01x06_Socket, symbol Connector:Conn_01x06_Socket
